File: hw/adb_kvm_0p1/VintageKVM.kicad_pcb (KiCad board)
At the start: 2 copper layers, 200 x 73.6 mm, 178 parts, among them J1 Micro USB, J10 DE15_Receptacle_HighDensity_M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, J12 DE15_Receptacle_HighDensity_M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, J14 DE15_Receptacle_HighDensity_M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, J2 Conn_01x20_Pin, J3 Conn_02x10_Odd_Even, J4 Conn_01x20_Pin, J6 DE15_Receptacle_HighDensity_M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, J8 DE15_Receptacle_HighDensity_M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, Q1 BSS138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

Commit message: fixed selection logic
Parts:
- added REF**: DSUB-15_Male_EdgeMount_P2.77mm, Connector_Dsub:DSUB-15_Male_EdgeMount_P2.77mm, F.Cu at (-78.7, 68.6)
